Commit message: Update test_robot.urdf

File: test_robot.urdf (robot description, URDF)
Before this commit: robot  test_urdf , 3 links, 2 joints
Joints:
- joint base_to_link_2: origin xyz=0.6 0.0 0.0 rpy=0.0 0.0 0.0 -> xyz=0.0 0.0 0.6 rpy=0.0 0.5 0.0; type revolute -> fixed
- joint link_2_to_camera: child camera_link  -> camera_link; origin xyz=0.6 0.0 0.0 rpy=0.0 0.0 0.0 -> xyz=0.0 0.0 0.6 rpy=0.0 0.0 0.0
